File: kicad/sensor-net-gateway-bl651/power.sch (KiCad schematic (older format))
At the start: 8 parts

Commit message: routing snapshot
Changed lines of the file:
@@
 Connection ~ 7800 3750
 Wire Wire Line
-	4300 4350 4500 4350
-Text HLabel 4400 4350 3    50   Input ~ 0
-GND
+	4300 4350 4400 4350
+$Comp
+L power:GND #PWR?
+U 1 1 5F959CCD
+P 4400 4350
+F 0 "#PWR?" H 4400 4100 50  0001 C CNN
+F 1 "GND" H 4405 4177 50  0000 C CNN
+F 2 "" H 4400 4350 50  0001 C CNN
+F 3 "" H 4400 4350 50  0001 C CNN
+	1    4400 4350
+	1    0    0    -1
+$EndComp
+Connection ~ 4400 4350
+Wire Wire Line
+	4400 4350 4500 4350
 $EndSCHEMATC
