File: kicad/sensor-net-gateway-bl651/usb.sch (KiCad schematic (older format))
At the start: 0 parts

Commit message: added power and usb2uart
Parts:
- added C1, C21, C5, C6: 0.1µF, Capacitor_SMD:C_0603_1608Metric, symbol Device:C
- added C11: 10nF, Capacitor_SMD:C_0603_1608Metric, symbol Device:C
- added C2, C3: 47pF, Capacitor_SMD:C_0603_1608Metric, symbol Device:C
- added C4: 4.7µF, WurthElektronik:865080640004, symbol Device:CP
- added FB1: Ferrite_Bead, Capacitor_SMD:C_0805_2012Metric, symbol HH_Laird:Ferrite_Bead
- added R1, R2: 27R, Resistor_SMD:R_0603_1608Metric, symbol Device:R
- added U1: USB_micro_ab, HH_Molex:MOLEX_USB_MICRO_0475890001, symbol HH_Molex:USB_micro_ab
- added U2: USBLC6-2SC6, HH_STMicroelectronics:USBLC6-2SC6_SOT-23-6, symbol HH_STMicroelectronics:USBLC6-2SC6
- added U3: FT230XQ, Package_DFN_QFN:QFN-16-1EP_4x4mm_P0.65mm_EP2.1x2.1mm, symbol Interface_USB:FT230XQ
Connections:
- new net: C2.1, R1.2, U2.3 (IN/USBDM)
- new net: C3.1, R2.2, U2.1 (IN/USBDP)
- new net: R2.1, U3.6 (USBDP)
- new net: R1.1, U3.7 (USBDM)
- new net: C4.1, C6.2, FB1.2, U3.10 (VCC)
- new net: C5.1, U3.8 (3V3OUT), U3.9 (~RESET)
- new net: U1.2 (DM), U2.4 (OUT/USBDM)
- new net: U1.3 (DP), U2.6 (OUT/USBDP)
- new net 3V0: C21.1, U3.1 (VCCIO)
- new net FTDI_DIO0: U3.12 (CBUS0)
- new net FTDI_DIO1: U3.11 (CBUS1)
- new net FTDI_DIO2: U3.5 (CBUS2)
- new net FTDI_DIO3: U3.14 (CBUS3)
- new net GND: C1.2, C11.2, C2.2, C21.2, C3.2, C4.2, C5.2, C6.1, U1.5 (GND), U2.2 (GND), U3.13 (GND), U3.17 (GND), U3.3 (GND)
- new net UART.CTS: U3.4 (~CTS)
- new net UART.RTS: U3.16 (~RTS)
- new net UART.RX: U3.2 (RXD)
- new net UART.TX: U3.15 (TXD)
- new net VBUS: C1.1, C11.1, FB1.1, U1.1 (VBUS), U2.5 (V_BUS)
- no-connect marks 0 -> 1
Other:
- note added: "ESD Protection"
- note added: "USB Connector"
- note added: "USB to UART"
