File: kicad/sensor-net-gateway-bl651/usb.sch (KiCad schematic (older format))
At the start: 14 parts, among them U1 USB_micro_ab, U2 USBLC6-2SC6, U3 FT230XQ

Commit message: started layout
Parts:
- C4: footprint WurthElektronik:865080640004 -> HH_WurthElektronik:865080640004
Changed lines of the file:
@@
 $Descr A4 11693 8268
 encoding utf-8
-Sheet 4 4
+Sheet 4 5
 Title ""
 Date ""
@@
 F 0 "C4" H 7232 2654 50  0000 R CNN
 F 1 "4.7µF" H 7232 2745 50  0000 R CNN
-F 2 "WurthElektronik:865080640004" H 7388 2550 50  0001 C CNN
+F 2 "HH_WurthElektronik:865080640004" H 7388 2550 50  0001 C CNN
 F 3 "https://katalog.we-online.de/pbs/datasheet/865080640004.pdf" H 7350 2700 50  0001 C CNN
 F 4 "732-8449-1-ND" H 7350 2700 50  0001 C CNN "DigiKey_PartNumber"

Commit message: routing snapshot
Connections:
- net D_N: now reaches U1.2 (DM), U2.4 (OUT/USBDM)
- net D_P: now reaches U1.3 (DP), U2.6 (OUT/USBDP)
Changed lines of the file:
@@
 $EndComp
 Wire Wire Line
-	4000 4400 4000 4250
+	4000 4400 4000 4350
 $Comp
 L Device:C C2
@@
 Wire Wire Line
 	9200 2700 9250 2700
-Text HLabel 9250 2100 2    50   Input ~ 0
-GND
-Text HLabel 9250 2700 2    50   Input ~ 0
-GND
-Text HLabel 8350 4600 3    50   Input ~ 0
-GND
-Text HLabel 7600 4800 3    50   Input ~ 0
-GND
-Text HLabel 6900 4700 3    50   Input ~ 0
-GND
-Text HLabel 4000 4400 3    50   Input ~ 0
-GND
-Text HLabel 6550 2500 0    50   Input ~ 0
-GND
 Wire Wire Line
 	7600 3250 7600 3650
@@
 Wire Wire Line
 	4000 3950 4550 3950
-Text HLabel 5550 3650 2    50   Input ~ 0
-GND
-Text HLabel 3600 3450 2    50   Input ~ 0
-GND
 Wire Wire Line
 	3600 3750 3950 3750
@@
 Text HLabel 9050 3950 2    50   Input ~ 0
 FTDI_DIO2
+Text Label 3850 3650 1    50   ~ 0
+D_P
+Text Label 3850 3750 3    50   ~ 0
+D_N
+$Comp
+L power:GND #PWR?
+U 1 1 5F95B5C0
+P 8350 4600
+F 0 "#PWR?" H 8350 4350 50  0001 C CNN
+F 1 "GND" H 8355 4427 50  0000 C CNN
+F 2 "" H 8350 4600 50  0001 C CNN
+F 3 "" H 8350 4600 50  0001 C CNN
+	1    8350 4600
+	1    0    0    -1
+$EndComp
+$Comp
+L power:GND #PWR?
+U 1 1 5F95B8AC
+P 7600 4800
+F 0 "#PWR?" H 7600 4550 50  0001 C CNN
+F 1 "GND" H 7605 4627 50  0000 C CNN
+F 2 "" H 7600 4800 50  0001 C CNN
+F 3 "" H 7600 4800 50  0001 C CNN
+	1    7600 4800
+	1    0    0    -1
+$EndComp
+$Comp
+L power:GND #PWR?
+U 1 1 5F95BDE8
+P 6900 4700
+F 0 "#PWR?" H 6900 4450 50  0001 C CNN
+F 1 "GND" H 6905 4527 50  0000 C CNN
+F 2 "" H 6900 4700 50  0001 C CNN
+F 3 "" H 6900 4700 50  0001 C CNN
+	1    6900 4700
+	1    0    0    -1
+$EndComp
+$Comp
+L power:GND #PWR?
+U 1 1 5F95C56F
+P 4000 4400
+F 0 "#PWR?" H 4000 4150 50  0001 C CNN
+F 1 "GND" H 4005 4227 50  0000 C CNN
+F 2 "" H 4000 4400 50  0001 C CNN
+F 3 "" H 4000 4400 50  0001 C CNN
+	1    4000 4400
+	1    0    0    -1
+$EndComp
+Wire Wire Line
+	3600 3450 3700 3450
+Wire Wire Line
+	3700 3450 3700 4350
+Wire Wire Line
+	3700 4350 4000 4350
+Connection ~ 4000 4350
+Wire Wire Line
+	4000 4350 4000 4250
+Wire Wire Line
+	5650 4350 5650 3650
+Wire Wire Line
+	5650 3650 5550 3650
+Wire Wire Line
+	4000 4350 5650 4350
+$Comp
+L power:GND #PWR?
+U 1 1 5F962756
+P 6550 2500
+F 0 "#PWR?" H 6550 2250 50  0001 C CNN
+F 1 "GND" H 6555 2327 50  0000 C CNN
+F 2 "" H 6550 2500 50  0001 C CNN
+F 3 "" H 6550 2500 50  0001 C CNN
+	1    6550 2500
+	1    0    0    -1
+$EndComp
+$Comp
+L power:GND #PWR?
+U 1 1 5F963429
+P 9250 2850
+F 0 "#PWR?" H 9250 2600 50  0001 C CNN
+F 1 "GND" H 9255 2677 50  0000 C CNN
+F 2 "" H 9250 2850 50  0001 C CNN
+F 3 "" H 9250 2850 50  0001 C CNN
+	1    9250 2850
+	1    0    0    -1
+$EndComp
+Wire Wire Line
+	9250 2100 9250 2700
+Wire Wire Line
+	9250 2700 9250 2850
+Connection ~ 9250 2700
 $EndSCHEMATC
